Commit message: got the state publisher connected with the inverse kinematics server. now the arm can move to the target set by the user.

File: robot_arm/urdf/model.urdf (robot description, URDF)
Before this commit: robot arm, 10 links, 9 joints
Links:
- added link end_effector
Joints:
- added joint link6_to_end_eff: type fixed, parent link6, child end_effector, origin xyz=0.5 0 0

Commit message: changed robot wrist to spherical type and changed length of link6 to 0.3 instead of 0.5

File: robot_arm/urdf/model.urdf (robot description, URDF)
Before this commit: robot arm, 11 links, 10 joints
Links:
- removed link l5_6_connector1
- removed link l5_6_connector2
- link link5: geometry visual cylinder length=.4 radius=0.2
- link link6: geometry visual cylinder length=.3 radius=0.1
Joints:
- removed joint connector1_to_connector2
- removed joint connector2_to_link6
- removed joint link5_to_connector1
- added joint link5_to_link6: type revolute, parent link5, child link6, origin xyz=0.3 0 0, axis 0 1 0, limit lower=-3.14 upper=3.14 effort=10 velocity=1
- joint link4_to_link5: axis 0 0 1 -> (none); limit lower=-3.14 upper=3.14 effort=10 velocity=1 -> (none); origin xyz=0.5 0 0 -> xyz=0.1 0 0; type revolute -> fixed
- joint link6_to_end_eff: axis (none) -> 1 0 0; limit (none) -> lower=-3.14 upper=3.14 effort=10 velocity=1; origin xyz=0.5 0 0 -> xyz=0.3 0 0; type fixed -> revolute

Commit message: added inverse kinematics for the spherical wrist. did some testing and its slightly inconsistent. could also be because inverse kinematics didn't give precise angles. need to change the arm links so thee workspace is better

File: robot_arm/urdf/model.urdf (robot description, URDF)
Before this commit: robot arm, 9 links, 8 joints
Links:
- link link4: geometry 
Joints:
- joint link4_to_link5: origin xyz=0.1 0 0 -> xyz=0 0 0

Commit message: changed the length of the links and added xacro in the URDF. tried to fix the wrist ik. maybe need to change rotation axis and order?

File: robot_arm/urdf/model.urdf (robot description, URDF)
Before this commit: robot arm, 9 links, 8 joints
Links:
- removed link link6
- added link link5_roll
- link base_link: geometry visual cylinder length=${base_len} radius=0.2
- link link1: geometry visual cylinder length=${l1_len} radius=0.1
- link link2: geometry visual cylinder length=${l2_len} radius=0.1
- link link3: geometry visual cylinder length=${l3_len} radius=0.1
- link link4: geometry visual cylinder length=${l4_width} radius=${l4_len/2}
- link link5: geometry visual cylinder length=${l5_len} radius=0.1
Joints:
- removed joint link4_to_link5
- removed joint link5_to_link6
- removed joint link6_to_end_eff
- added joint link4_to_link5_pitch: type revolute, parent link4, child link5, origin xyz=${l4_len} 0 0 rpy=0 0 0, axis 0 1 0, limit lower=-3.14 upper=3.14 effort=10 velocity=1
- added joint link4_to_link5_roll: type revolute, parent link5, child link5_roll, origin xyz=0 0 0 rpy=0 0 0, axis 1 0 0, limit lower=-3.14 upper=3.14 effort=10 velocity=1
- added joint link5_to_end: type fixed, parent link5_roll, child end_effector, origin xyz=${l5_len} 0 0 rpy=0 0 0
- joint base_to_link1: origin xyz=0 0 0.5 rpy=0 0 0 -> xyz=0 0 ${base_len} rpy=0 0 0
- joint link1_to_link2: origin xyz=0 0 0.5 rpy=0 0 0 -> xyz=0 0 ${l1_len} rpy=0 0 0
- joint link2_to_link3: origin xyz=0.5 0 0 -> xyz=${l2_len} 0 0 rpy=0 0 0
- joint link3_to_link4: origin xyz=0.5 0 0 -> xyz=${l3_len} 0 0 rpy=0 0 0

Commit message: added some initial constraints for joint angles. added collision and inertial properties for the URDF

File: robot_arm/urdf/model.urdf (robot description, URDF)
Before this commit: robot arm, 9 links, 8 joints
Links:
- link base_link: geometry collision cylinder length=${base_len} radius=${base_radius}; visual cylinder length=${base_len} radius=${base_radius}
- link link1: mass None -> 10; geometry collision cylinder length=${l1_len} radius=${l1_radius}; visual cylinder length=${l1_len} radius=${l1_radius}
- link link2: mass None -> 10; geometry collision cylinder length=${l2_len} radius=${l2_radius}; visual cylinder length=${l2_len} radius=${l1_radius}
- link link3: mass None -> 10; geometry collision cylinder length=${l3_len} radius=${l3_radius}; visual cylinder length=${l3_len} radius=${l3_radius}
- link link4: mass None -> 10; geometry collision cylinder length=${l4_width} radius=${l4_len/2}; visual cylinder length=${l4_width} radius=${l4_len/2}
- link link5: mass None -> 10; geometry collision cylinder length=${l5_len} radius=${l5_radius}; visual cylinder length=${l5_len} radius=${l5_radius}
- link link5_roll: mass None -> 10

Commit message: integrated mesh files into urdf model and changed joint len variables

File: robot_arm/urdf/model.urdf (robot description, URDF)
Before this commit: robot arm, 9 links, 8 joints
Links:
- link base_link: geometry visual mesh filename=package://robot_arm/meshes/base.stl scale=0.01 0.01 0.01
- link link1: geometry visual mesh filename=package://robot_arm/meshes/link1.stl scale=0.01 0.01 0.01
- link link2: geometry visual mesh filename=package://robot_arm/meshes/link2.stl scale=0.01 0.01 0.01
- link link3: geometry collision mesh filename=package://robot_arm/meshes/link3.stl scale=0.01 0.01 0.01; visual mesh filename=package://robot_arm/meshes/link3.stl scale=0.01 0.01 0.01
- link link4: geometry collision mesh filename=package://robot_arm/meshes/link4.stl scale=0.01 0.01 0.01; visual mesh filename=package://robot_arm/meshes/link4.stl scale=0.01 0.01 0.01
- link link5: geometry collision mesh filename=package://robot_arm/meshes/link5.stl scale=0.01 0.01 0.01; visual mesh filename=package://robot_arm/meshes/link5.stl scale=0.01 0.01 0.01
Joints:
- joint axis_to_base: origin (none) -> xyz=0 0 0 rpy=0 0 0
- joint base_to_link1: origin xyz=0 0 ${base_len} rpy=0 0 0 -> xyz=0 0 0.55 rpy=0 0 0
- joint link1_to_link2: origin xyz=0 0 ${l1_len} rpy=0 0 0 -> xyz=0 0 0 rpy=0 0 0
- joint link2_to_link3: origin xyz=${l2_len} 0 0 rpy=0 0 0 -> xyz=0.75 0 0.2 rpy=0 0 0
- joint link3_to_link4: origin xyz=${l3_len} 0 0 rpy=0 0 0 -> xyz=0.85 0 0 rpy=0 0 0
- joint link4_to_link5_pitch: origin xyz=${l4_len} 0 0 rpy=0 0 0 -> xyz=0.3 0 0 rpy=0 0 0
- joint link4_to_link5_roll: origin xyz=0 0 0 rpy=0 0 0 -> xyz=0 0 -0.40 rpy=0 0 0
- joint link5_to_end: origin xyz=0 0 -${l5_len} rpy=0 0 0 -> xyz=0 0 0 rpy=0 0 0
